Commit message: alpha_urdf done

File: alpha_description/urdf/chassis/alpha_base.transmission.xacro (robot description, xacro)
@@ -15,7 +15,10 @@
   <xacro:macro name="alpha_caster_transmission" params="suffix">
     <transmission type="alpha_mechanism_model/SimpleTransmission" name="${suffix}_rotation_trans">
-      <actuator name="${suffix}_rotation_motor" />
-      <joint name="${suffix}_rotation_joint" />
-      <mechanicalReduction>${-1 * 624/35 * 80/18}</mechanicalReduction>
+      <actuator name="${suffix}_rotation_motor">
+        <mechanicalReduction>${-1 * 624/35 * 80/18}</mechanicalReduction>
+      </actuator>
+      <joint name="${suffix}_rotation_joint">
+        <hardwareInterface>EffortJointInterface</hardwareInterface>
+      </joint>
     </transmission>
   </xacro:macro>

File: alpha_description/urdf/chassis/alpha_base.urdf.xacro (robot description, xacro)
@@ -1,46 +1,178 @@
 <?xml version="1.0"?>
-<robot xmlns:xacro="http://ros.org/wiki/xacro">
-  <xacro:property name="base_link_wheel_seperation" value="0.30" />
-  <xacro:property name="base_link_wheel_diameter" value="0.09" />
-  <xacro:property name="base_link_wheel_torque" value="0.01" />
-  <xacro:macro name="alpha_wheel_gazebo" params="suffix parent">
-    <gazebo reference="${parent}_${suffix}_wheel_link">
-      <mu1 value="1.0" />
-      <mu2 value="1.0" />
-      <kp  value="1000000.0" />
-      <kd  value="100.0" />
-      <maxVel  value="1.0" />
-      <minDepth  value="0.001" />
-    </gazebo>
+<robot xmlns:sensor="http://playerstage.sourceforge.net/gazebo/xmlschema/#sensor"
+       xmlns:controller="http://playerstage.sourceforge.net/gazebo/xmlschema/#controller"
+       xmlns:interface="http://ros.org/wiki/xacro"
+       xmlns:xacro="http://ros.org/wiki/xacro">
+  <xacro:include filename="$(find alpha_description)/urdf/chassis/alpha_base.gazebo.xacro" />
+  <xacro:include filename="$(find alpha_description)/urdf/chassis/alpha_base.transmission.xacro" />
+  <!-- DATA SOURCES -->
+  <!-- all link geometry sizes are obtained from Function provided CAD model unless stated otherwise -->
+  <!-- all simplified collision geometry are hand approximated from CAD model, sometimes from respective bounding boxes -->
+  <xacro:property name="M_PI" value="3.1415926535897931" />
+  <xacro:property name="caster_offset_x" value="0.115" />
+  <xacro:property name="caster_offset_y" value="0.0" />
+  <xacro:property name="caster_offset_z" value="0.007" />
+  <xacro:property name="caster_mass" value="0.01" />
+  <xacro:property name="wheel_offset_z" value="0.026" />
+  <xacro:property name="wheel_length" value="0.0206" />
+  <xacro:property name="wheel_radius" value="0.0350" />
+  <xacro:property name="wheel_mass" value="0.01" />
+  <xacro:property name="caster_wheel_offset_y" value="0.28" />
+  <xacro:property name="base_cg_x" value="0.001" />
+  <xacro:property name="base_cg_y" value="0.0" />
+  <xacro:property name="base_cg_z" value="-0.034" />
+  <xacro:property name="base_mass" value="2.4" />
+  <!-- simplified box collision geometry for base -->
+  <xacro:property name="base_collision_length" value="0.10938" />
+  <xacro:property name="base_collision_radius" value="0.178" />
+  <xacro:property name="base_collision_z" value="0.05949" />
+  <!-- Macro for aplha wheel (right/left)-->
+  <!-- in typical convention param "reflect" equals +-1 to distinguish left from righ-->
+  <xacro:macro name="alpha_wheel" params="suffix parent reflect">
+    <joint name="${parent}_${suffix}_wheel_joint" type="continuous">
+      <axis xyz="0 0 1" />
+      <limit effort="18" velocity="1.5"/>
+      <safety_controller  k_velocity="1" />
+      <dynamics damping="1.0" friction="0.0" />
+      <origin xyz="0 ${reflect * caster_wheel_offset_y} ${wheel_offset_z}" rpy="${-M_PI/2} 0 0" />
+      <parent link="${parent}_rotation_link"/>
+      <child link="${parent}_${suffix}_wheel_link"/>
+    </joint>
+    <link name="${parent}_${suffix}_wheel_link">
+      <inertial>
+        <mass value="${wheel_mass}" />
+        <origin xyz="0 0 0" />
+        <inertia  ixx="0.001" ixy="0.0" ixz="0.0"
+                  iyy="0.001" iyz="0.0"
+                  izz="0.001" />
+      </inertial>
+      <visual>
+        <origin xyz="0 0 0" rpy="0 0 0" />
+        <geometry>
+          <mesh filename="package://alpha_description/meshes/chassis/wheel.dae" />
+        </geometry>
+        <material name="Wheel_${suffix}" />
+      </visual>
+      <collision>
+        <origin xyz="0 0 0" rpy="${M_PI/2} 0 0" /> <!-- rotation because cyl. geom primitive has symmetry axis in +x direction -->
+        <geometry>
+          <cylinder radius="${wheel_radius}" length="${wheel_length}" />
+        </geometry>
+      </collision>
+    </link>
+    <!-- extensions -->
+    <xacro:alpha_wheel_gazebo parent="${parent}" suffix="${suffix}" />
+    <xacro:alpha_wheel_transmission parent="${parent}" suffix="${suffix}" reflect="${reflect}" />
   </xacro:macro>
-  <xacro:macro name="alpha_caster_gazebo" params="suffix">
-    <gazebo reference="${suffix}_caster_rotation_link">
-      <mu1 value="0.0" />
-      <mu2 value="0.0" />
-      <kp value="1000000.0" />
-      <kd value="100.0" />
-      <minDepth value="0.001" />
-      <maxVel value="1.0" />
-    </gazebo>
+  <!-- Macro for alpha caster hub only -->
+  <xacro:macro name="alpha_caster_hub" params="suffix parent *origin ref_position" >
+    <joint name="${suffix}_rotation_joint" type="continuous">
+      <axis xyz="0 0 1" />
+      <origin xyz="${caster_offset_x} 0 ${caster_offset_z}" rpy="${-M_PI/2} 0 0"/>
+      <limit effort="18" velocity="1.5"/>
+      <safety_controller  k_velocity="1" />
+      <calibration rising="${ref_position}" />
+      <dynamics damping="1.0" friction="0.0" />
+      <xacro:insert_block name="origin" />
+      <parent link="${parent}"/>
+      <child link="${suffix}_rotation_link" />
+    </joint>
+    <link name="${suffix}_rotation_link">
+      <inertial>
+        <mass value="${caster_mass}"/>
+        <origin xyz="0 0 0" />
+        <inertia ixx="0.001" ixy="0.0" ixz="0.0"
+                 iyy="0.001" iyz="0.0"
+                 izz="0.001" />
+      </inertial>
+      <visual>
+        <origin xyz="0 0 0" rpy="0 0 0" />
+        <geometry>
+          <mesh filename="package://alpha_description/meshes/chassis/caster.stl" />
+        </geometry>
+        <material name="Caster" />
+      </visual>
+      <collision>
+        <origin xyz="0 0 0" rpy="0 0 0" />
+        <geometry>
+          <mesh filename="package://alpha_description/meshes/chassis/caster_L.stl" />
+        </geometry>
+      </collision>
+    </link>
+    <!-- extensions -->
+    <xacro:alpha_caster_transmission suffix="${suffix}" />
   </xacro:macro>
-  <xacro:macro name="alpha_base_gazebo" params="name">
-    <gazebo reference="${name}_link">
-      <selfCollide>false</selfCollide>
-    </gazebo>
-    <gazebo>
-      <plugin name="differential_drive_controller" filename="libgazebo_ros_diff_drive.so">
-        <alwaysOn>true</alwaysOn>
-        <leftJoint>${name}_link_right_wheel_joint</leftJoint>
-        <rightJoint>${name}_link_left_wheel_joint</rightJoint>
-        <wheel_separation>${${name}_link_wheel_seperation}</wheel_separation>
-        <wheel_diameter>${${name}_link_wheel_diameter}</wheel_diameter>
-        <torque>${${name}_link_wheel_torque}</torque>
-        <publish_tf>1</publish_tf>
-        <commandTopic>cmd_vel</commandTopic>
-        <odometryTopic>odom</odometryTopic>
-        <odometryFrame>odom</odometryFrame>
-        <robotBaseFrame>base_footprint</robotBaseFrame>
-      </plugin>
-	  </gazebo>
+  <!-- The xacro macro xacro:alpha_caster contains: caster and wheels -->
+  <xacro:macro name="alpha_caster" params="suffix parent *origin ref_position">
+    <xacro:alpha_caster_hub parent="${parent}" suffix="${suffix}_caster" ref_position="${ref_position}" >
+      <xacro:insert_block name="origin" />
+    </xacro:alpha_caster_hub>
+    <!-- wheel macros -->
+    <xacro:alpha_wheel parent="${suffix}_caster" suffix="l" reflect="1" />
+    <xacro:alpha_wheel parent="${suffix}_caster" suffix="r" reflect="-1" />
+    <!-- extensions -->
+    <xacro:alpha_caster_gazebo suffix="${suffix}" />
+  </xacro:macro>
+  <!-- The xacro macro xacro:alpha_base contains: base, caster and wheels -->
+  <xacro:macro name="alpha_base" params="name">
+    <link name="${name}_link">
+      <inertial>
+        <mass value="${base_mass}" />
+        <origin xyz="${base_cg_x} ${base_cg_y} ${base_cg_z}" />
+        <inertia ixx="0.019995" ixy="0.0" ixz="0.0"
+                 iyy="0.019995" iyz="0.0"
+                 izz="0.03675" />
+      </inertial>
+      <visual>
+        <origin xyz="0 0 0" rpy="0 0 0" />
+        <geometry>
+          <mesh filename="package://alpha_description/meshes/chassis/base_plate.dae" />
+        </geometry>
+        <material name="White" />
+      </visual>
+      <collision>
+        <origin xyz="0 0 0" rpy="0 0 0" />
+        <geometry>
+          <cylinder radius="${base_collision_radius}" length="${base_collision_length}" />
+        </geometry>
+      </collision>
+    </link>
+    <!-- base_footprint is a fictitious link(frame) that is on the ground right below base_link origin,
+         navigation stack dedpends on this frame -->
+    <link name="${name}_footprint">
+      <inertial>
+        <mass value="1.0" />
+        <origin xyz="0 0 0" />
+        <inertia ixx="0.019995" ixy="0.0" ixz="0.0"
+                 iyy="0.019995" iyz="0.0"
+                 izz="0.03675" />
+      </inertial>
+      <visual>
+        <origin xyz="0 0 0" rpy="0 0 0" />
+        <geometry>
+          <box size="0.01 0.01 0.01" />
+        </geometry>
+        <material name="White" />
+      </visual>
+      <collision>
+        <!-- represent base collision with a simple rectangular model, positioned by base_size_z s.t. top
+             surface of the collision box matches the top surface of the alpha base -->
+        <origin xyz="0 0 ${0.051+base_collision_z/2}" rpy="0 0 0" />
+        <geometry>
+          <box size="0.001 0.001 0.001" />
+        </geometry>
+      </collision>
+    </link>
+    <joint name="${name}_footprint_joint" type="fixed">
+      <origin xyz="0 0 0.051" rpy="0 0 0" />
+      <child link="${name}_link" />
+      <parent link="${name}_footprint"/>
+    </joint>
+    <!-- caster macro -->
+    <xacro:alpha_caster suffix="fl" parent="${name}_link" ref_position="${- M_PI/4}" >
+      <origin xyz="${caster_offset_x} ${caster_offset_y} ${caster_offset_z}" rpy="0 0 0" />
+    </xacro:alpha_caster>
+    <!-- gazebo extensions -->
+    <xacro:alpha_base_gazebo name="${name}" />
   </xacro:macro>
 </robot>
