Commit message: rviz config added

File: alpha_description/urdf/chassis/alpha_base.urdf.xacro (robot description, xacro)
@@ -69,5 +69,5 @@
     <joint name="${suffix}_rotation_joint" type="continuous">
       <axis xyz="0 0 1" />
-      <origin xyz="${caster_offset_x} 0 ${caster_offset_z}" rpy="${-M_PI/2} 0 0"/>
+      <origin xyz="${caster_offset_x} 0 ${caster_offset_z}" rpy="0 0 0"/>
       <limit effort="18" velocity="1.5"/>
       <safety_controller  k_velocity="1" />
@@ -170,5 +170,5 @@
     </joint>
     <!-- caster macro -->
-    <xacro:alpha_caster suffix="fl" parent="${name}_link" ref_position="${- M_PI/4}" >
+    <xacro:alpha_caster suffix="fl" parent="${name}_link" ref_position="0" >
       <origin xyz="${caster_offset_x} ${caster_offset_y} ${caster_offset_z}" rpy="0 0 0" />
     </xacro:alpha_caster>

Commit message: transformations set correctly

File: alpha_description/urdf/chassis/alpha_base.urdf.xacro (robot description, xacro)
@@ -6,20 +6,23 @@
   <xacro:include filename="$(find alpha_description)/urdf/chassis/alpha_base.gazebo.xacro" />
   <xacro:include filename="$(find alpha_description)/urdf/chassis/alpha_base.transmission.xacro" />
+  <xacro:include filename="$(find alpha_description)/urdf/materials.urdf.xacro" />
   <!-- DATA SOURCES -->
   <!-- all link geometry sizes are obtained from Function provided CAD model unless stated otherwise -->
   <!-- all simplified collision geometry are hand approximated from CAD model, sometimes from respective bounding boxes -->
   <xacro:property name="M_PI" value="3.1415926535897931" />
-  <xacro:property name="caster_offset_x" value="0.115" />
+  <xacro:property name="caster_offset_x" value="0.0" />
   <xacro:property name="caster_offset_y" value="0.0" />
-  <xacro:property name="caster_offset_z" value="0.007" />
+  <xacro:property name="caster_offset_z" value="-0.02" />
   <xacro:property name="caster_mass" value="0.01" />
-  <xacro:property name="wheel_offset_z" value="0.026" />
+  <xacro:property name="caster_collision_length" value="0.0176" />
+  <xacro:property name="caster_collision_radius" value="0.017" />
+  <xacro:property name="wheel_offset_y" value="0.14" />
+  <xacro:property name="wheel_offset_z" value="0.0" />
+  <xacro:property name="wheel_mass" value="0.01" />
   <xacro:property name="wheel_length" value="0.0206" />
   <xacro:property name="wheel_radius" value="0.0350" />
-  <xacro:property name="wheel_mass" value="0.01" />
-  <xacro:property name="caster_wheel_offset_y" value="0.28" />
-  <xacro:property name="base_cg_x" value="0.001" />
+  <xacro:property name="base_cg_x" value="0.0" />
   <xacro:property name="base_cg_y" value="0.0" />
-  <xacro:property name="base_cg_z" value="-0.034" />
+  <xacro:property name="base_cg_z" value="0.065" />
   <xacro:property name="base_mass" value="2.4" />
   <!-- simplified box collision geometry for base -->
@@ -35,5 +38,5 @@
       <safety_controller  k_velocity="1" />
       <dynamics damping="1.0" friction="0.0" />
-      <origin xyz="0 ${reflect * caster_wheel_offset_y} ${wheel_offset_z}" rpy="${-M_PI/2} 0 0" />
+      <origin xyz="0 ${reflect * wheel_offset_y} ${wheel_offset_z}" rpy="${-M_PI/2} 0 0" />
       <parent link="${parent}_rotation_link"/>
       <child link="${parent}_${suffix}_wheel_link"/>
@@ -67,12 +70,6 @@
   <!-- Macro for alpha caster hub only -->
   <xacro:macro name="alpha_caster_hub" params="suffix parent *origin ref_position" >
-    <joint name="${suffix}_rotation_joint" type="continuous">
-      <axis xyz="0 0 1" />
-      <origin xyz="${caster_offset_x} 0 ${caster_offset_z}" rpy="0 0 0"/>
-      <limit effort="18" velocity="1.5"/>
-      <safety_controller  k_velocity="1" />
-      <calibration rising="${ref_position}" />
-      <dynamics damping="1.0" friction="0.0" />
-      <xacro:insert_block name="origin" />
+    <joint name="${suffix}_rotation_joint" type="fixed">
+      <origin xyz="${caster_offset_x} ${caster_offset_y} ${caster_offset_z}" rpy="0 0 ${-M_PI/2}"/>
       <parent link="${parent}"/>
       <child link="${suffix}_rotation_link" />
@@ -86,15 +83,8 @@
                  izz="0.001" />
       </inertial>
-      <visual>
-        <origin xyz="0 0 0" rpy="0 0 0" />
-        <geometry>
-          <mesh filename="package://alpha_description/meshes/chassis/caster.stl" />
-        </geometry>
-        <material name="Caster" />
-      </visual>
       <collision>
         <origin xyz="0 0 0" rpy="0 0 0" />
         <geometry>
-          <mesh filename="package://alpha_description/meshes/chassis/caster_L.stl" />
+          <cylinder length="${caster_collision_length}" radius="${caster_collision_radius}"/>
         </geometry>
       </collision>
@@ -119,5 +109,5 @@
       <inertial>
         <mass value="${base_mass}" />
-        <origin xyz="${base_cg_x} ${base_cg_y} ${base_cg_z}" />
+        <origin xyz="0 0 0" />
         <inertia ixx="0.019995" ixy="0.0" ixz="0.0"
                  iyy="0.019995" iyz="0.0"
@@ -125,5 +115,5 @@
       </inertial>
       <visual>
-        <origin xyz="0 0 0" rpy="0 0 0" />
+        <origin xyz="0 0 -0.095" rpy="0 0 0" />
         <geometry>
           <mesh filename="package://alpha_description/meshes/chassis/base_plate.dae" />
@@ -158,5 +148,5 @@
         <!-- represent base collision with a simple rectangular model, positioned by base_size_z s.t. top
              surface of the collision box matches the top surface of the alpha base -->
-        <origin xyz="0 0 ${0.051+base_collision_z/2}" rpy="0 0 0" />
+        <origin xyz="0 0 ${base_collision_z/2}" rpy="0 0 0" />
         <geometry>
           <box size="0.001 0.001 0.001" />
@@ -165,10 +155,10 @@
     </link>
     <joint name="${name}_footprint_joint" type="fixed">
-      <origin xyz="0 0 0.051" rpy="0 0 0" />
+      <origin xyz="${base_cg_x} ${base_cg_y} ${base_cg_z}" rpy="0 0 0" />
+      <parent link="${name}_footprint"/>
       <child link="${name}_link" />
-      <parent link="${name}_footprint"/>
     </joint>
     <!-- caster macro -->
-    <xacro:alpha_caster suffix="fl" parent="${name}_link" ref_position="0" >
+    <xacro:alpha_caster suffix="fl" parent="${name}_link" ref_position="${- M_PI/4}" >
       <origin xyz="${caster_offset_x} ${caster_offset_y} ${caster_offset_z}" rpy="0 0 0" />
     </xacro:alpha_caster>

Commit message: tf tree added for urdf

File: alpha_description/urdf/chassis/alpha_base.urdf.xacro (robot description, xacro)
@@ -25,4 +25,5 @@
   <xacro:property name="base_cg_y" value="0.0" />
   <xacro:property name="base_cg_z" value="0.065" />
+  <xacro:property name="base_visual_offset" value="-0.095" />
   <xacro:property name="base_mass" value="2.4" />
   <!-- simplified box collision geometry for base -->
@@ -115,5 +116,5 @@
       </inertial>
       <visual>
-        <origin xyz="0 0 -0.095" rpy="0 0 0" />
+        <origin xyz="0 0 ${base_visual_offset}" rpy="0 0 0" />
         <geometry>
           <mesh filename="package://alpha_description/meshes/chassis/base_plate.dae" />

Commit message: right-left ambiguity in wheel

File: alpha_description/urdf/chassis/alpha_base.urdf.xacro (robot description, xacro)
@@ -39,5 +39,5 @@
       <safety_controller  k_velocity="1" />
       <dynamics damping="1.0" friction="0.0" />
-      <origin xyz="0 ${reflect * wheel_offset_y} ${wheel_offset_z}" rpy="${-M_PI/2} 0 0" />
+      <origin xyz="0 ${reflect * wheel_offset_y} ${wheel_offset_z}" rpy="${M_PI/2} 0 0" />
       <parent link="${parent}_rotation_link"/>
       <child link="${parent}_${suffix}_wheel_link"/>
@@ -96,10 +96,10 @@
   <!-- The xacro macro xacro:alpha_caster contains: caster and wheels -->
   <xacro:macro name="alpha_caster" params="suffix parent *origin ref_position">
-    <xacro:alpha_caster_hub parent="${parent}" suffix="${suffix}_caster" ref_position="${ref_position}" >
+    <xacro:alpha_caster_hub parent="${parent}" suffix="${suffix}" ref_position="${ref_position}" >
       <xacro:insert_block name="origin" />
     </xacro:alpha_caster_hub>
     <!-- wheel macros -->
-    <xacro:alpha_wheel parent="${suffix}_caster" suffix="l" reflect="1" />
-    <xacro:alpha_wheel parent="${suffix}_caster" suffix="r" reflect="-1" />
+    <xacro:alpha_wheel parent="${suffix}" suffix="left" reflect="-1" />
+    <xacro:alpha_wheel parent="${suffix}" suffix="right" reflect="1" />
     <!-- extensions -->
     <xacro:alpha_caster_gazebo suffix="${suffix}" />
