Commit message: kinect added

File: simulation_module/alpha_description/robots/alpha_bot.urdf.xacro (robot description, xacro)
@@ -8,5 +8,10 @@
   <!-- alpha base -->
   <xacro:include filename="$(find alpha_description)/urdf/chassis/alpha_base.urdf.xacro" />
+  <!-- kinect sensor -->
+  <xacro:include filename="$(find alpha_description)/urdf/sensors/kinect/kinect.urdf.xacro" />
   <!-- Now we can start using the macros included above to define the actual alpha -->
   <xacro:alpha_base name="base"/>
+  <xacro:kinect_camera name="kinect" parent="base_link">
+    <origin xyz="-0.137376 0 0.091746" rpy="0 0 0" />
+  </xacro:kinect_camera>
 </robot>

Commit message: position of kinect set

File: simulation_module/alpha_description/robots/alpha_bot.urdf.xacro (robot description, xacro)
@@ -13,5 +13,5 @@
   <xacro:alpha_base name="base"/>
   <xacro:kinect_camera name="kinect" parent="base_link">
-    <origin xyz="-0.137376 0 0.091746" rpy="0 0 0" />
+    <origin xyz="0 0.1575 0.181" rpy="0 0 ${M_PI/2}" />
   </xacro:kinect_camera>
 </robot>

Commit message: added hokoyu

File: simulation_module/alpha_description/robots/alpha_bot.urdf.xacro (robot description, xacro)
@@ -10,8 +10,16 @@
   <!-- kinect sensor -->
   <xacro:include filename="$(find alpha_description)/urdf/sensors/kinect/kinect.urdf.xacro" />
+  <!-- hokoyu laser sensor -->
+  <xacro:include filename="$(find alpha_description)/urdf/sensors/hokuyo_laser/hokuyo_lx30_laser.urdf.xacro" />
   <!-- Now we can start using the macros included above to define the actual alpha -->
+  <!-- alpha base -->
   <xacro:alpha_base name="base"/>
+  <!-- kinect sensor -->
   <xacro:kinect_camera name="kinect" parent="base_link">
     <origin xyz="0 0.1575 0.181" rpy="0 0 ${M_PI/2}" />
   </xacro:kinect_camera>
+  <!-- hokoyu laser sensor -->
+  <xacro:hokuyo_lx30_laser name="hokuyo" parent="base_link" ros_topic="tilt_scan" update_rate="40" min_angle="-1.3962634" max_angle="1.3962634" >
+    <origin xyz="0 0 0.03" rpy="0 0 0" />
+  </xacro:hokuyo_lx30_laser>
 </robot>

Commit message: kinect v2 and 360 models added

File: simulation_module/alpha_description/robots/alpha_bot.urdf.xacro (robot description, xacro)
@@ -9,5 +9,5 @@
   <xacro:include filename="$(find alpha_description)/urdf/chassis/alpha_base.urdf.xacro" />
   <!-- kinect sensor -->
-  <xacro:include filename="$(find alpha_description)/urdf/sensors/kinect/kinect.urdf.xacro" />
+  <xacro:include filename="$(find alpha_description)/urdf/sensors/kinect/v2/kinect.urdf.xacro" />
   <!-- hokoyu laser sensor -->
   <xacro:include filename="$(find alpha_description)/urdf/sensors/hokuyo_laser/hokuyo_lx30_laser.urdf.xacro" />

File: simulation_module/alpha_description/urdf/sensors/kinect/xbox360/kinect.urdf.xacro (robot description, xacro)
@@ -4,5 +4,5 @@
       xmlns:interface="http://ros.org/wiki/xacro"
       xmlns:xacro="http://ros.org/wiki/xacro">
-  <xacro:include filename="$(find alpha_description)/urdf/sensors/kinect/kinect.gazebo.xacro" />
+  <xacro:include filename="$(find alpha_description)/urdf/sensors/kinect/xbox360/kinect.gazebo.xacro" />
   <!-- Kinect Camera Location (Nominally 0) -->
   <xacro:property name="cal_kinect_x" value="0.0" />
@@ -29,5 +29,5 @@
         <origin xyz="0.0 0.012 0" rpy="0 0 0"/>
         <geometry>
-          <mesh filename="package://alpha_description/meshes/sensors/kinect/kinect.dae" scale="0.001 0.001 0.001" />
+          <mesh filename="package://alpha_description/meshes/sensors/kinect/xbox360/kinect.dae"/>
         </geometry>
       </visual>
@@ -35,5 +35,5 @@
         <origin xyz="0.0 0.012 0" rpy="0 0 0"/>
         <geometry>
-          <mesh filename="package://alpha_description/meshes/sensors/kinect/kinect.dae" scale="0.001 0.001 0.001" />
+          <mesh filename="package://alpha_description/meshes/sensors/kinect/xbox360/kinect.dae"/>
         </geometry>
       </collision>

Commit message: hokuyo mesh files added

File: simulation_module/alpha_description/robots/alpha_bot.urdf.xacro (robot description, xacro)
@@ -21,5 +21,5 @@
   <!-- hokoyu laser sensor -->
   <xacro:hokuyo_lx30_laser name="hokuyo" parent="base_link" ros_topic="tilt_scan" update_rate="40" min_angle="-1.3962634" max_angle="1.3962634" >
-    <origin xyz="0 0 0.03" rpy="0 0 0" />
+    <origin xyz="0 0 0.332" rpy="0 0 0" />
   </xacro:hokuyo_lx30_laser>
 </robot>

File: simulation_module/alpha_description/urdf/sensors/hokuyo_laser/hokuyo_lx30_laser.urdf.xacro (robot description, xacro)
@@ -10,13 +10,25 @@
       <xacro:insert_block name="origin" />
       <parent link="${parent}"/>
-      <child link="${name}_link"/>
+      <child link="${name}_frame"/>
     </joint>
-    <link name="${name}_link" type="laser">
-      <inertial>
-        <mass value="0.001" />
-        <origin xyz="0 0 0" rpy="0 0 0" />
-        <inertia ixx="0.0001" ixy="0" ixz="0" iyy="0.000001" iyz="0" izz="0.0001" />
-      </inertial>
-    </link>
+    <link name="${name}_frame">
+        <inertial>
+          <mass value="0.270" />
+          <origin xyz="0 0 0" rpy="0 0 0" />
+          <inertia ixx="2.632e-4" ixy="0" ixz="0" iyy="2.632e-4" iyz="0" izz="1.62e-4" />
+        </inertial>
+        <visual>
+          <origin xyz="0 0 0" rpy="0 0 0" />
+          <geometry>
+          <mesh filename="package://alpha_description/meshes/sensors/hokuyo_laser/hokuyo_utm_30lx.dae"/>
+        </geometry>
+        </visual>
+        <collision>
+          <origin xyz="0 0 -0.0115" rpy="0 0 0" />
+          <geometry>
+          <box size="0.058 0.058 0.087" />
+        </geometry>
+        </collision>
+      </link>
     <!-- gazebo extensions -->
     <xacro:hokuyo_lx30_laser_gazebo name="${name}" ros_topic="${ros_topic}" update_rate="${update_rate}" min_angle="${min_angle}" max_angle="${max_angle}" />

Commit message: hokuyo realigned

File: simulation_module/alpha_description/robots/alpha_bot.urdf.xacro (robot description, xacro)
@@ -21,5 +21,5 @@
   <!-- hokoyu laser sensor -->
   <xacro:hokuyo_lx30_laser name="hokuyo" parent="base_link" ros_topic="tilt_scan" update_rate="40" min_angle="-1.3962634" max_angle="1.3962634" >
-    <origin xyz="0 0 0.332" rpy="0 0 0" />
+    <origin xyz="0 0 0.332" rpy="0 0 ${M_PI/2}" />
   </xacro:hokuyo_lx30_laser>
 </robot>

Commit message: orientation of parts corrected

File: simulation_module/alpha_description/robots/alpha_bot.urdf.xacro (robot description, xacro)
@@ -17,9 +17,9 @@
   <!-- kinect sensor -->
   <xacro:kinect_camera name="kinect" parent="base_link">
-    <origin xyz="0 0.1575 0.181" rpy="0 0 ${M_PI/2}" />
+    <origin xyz="0 0.125 0.215" rpy="0 0 ${M_PI/2}" />
   </xacro:kinect_camera>
   <!-- hokoyu laser sensor -->
   <xacro:hokuyo_lx30_laser name="hokuyo" parent="base_link" ros_topic="base_scan" update_rate="40" min_angle="-1.3962634" max_angle="1.3962634" >
-    <origin xyz="0 0 0.332" rpy="0 0 ${M_PI/2}" />
+    <origin xyz="0 0 0.32" rpy="0 0 ${M_PI/2}" />
   </xacro:hokuyo_lx30_laser>
 </robot>

File: simulation_module/alpha_description/urdf/chassis/alpha_base.transmission.xacro (robot description, xacro)
@@ -9,5 +9,5 @@
       <actuator name="${parent}_${suffix}_wheel_motor" />
       <joint name="${parent}_${suffix}_wheel_joint" />
-      <mechanicalReduction>${reflect * 624/35 * 80/18}</mechanicalReduction>
+      <mechanicalReduction>${reflect * 1}</mechanicalReduction>
     </transmission>
   </xacro:macro>
@@ -15,8 +15,8 @@
   <xacro:macro name="alpha_caster_transmission" params="suffix">
     <transmission type="alpha_mechanism_model/SimpleTransmission" name="${suffix}_rotation_trans">
-      <actuator name="${suffix}_rotation_motor">
-        <mechanicalReduction>${-1 * 624/35 * 80/18}</mechanicalReduction>
+      <actuator name="${suffix}_rotation_caster">
+        <mechanicalReduction>1</mechanicalReduction>
       </actuator>
-      <joint name="${suffix}_rotation_joint">
+      <joint name="${suffix}_caster_joint">
         <hardwareInterface>EffortJointInterface</hardwareInterface>
       </joint>

File: simulation_module/alpha_description/urdf/chassis/alpha_base.urdf.xacro (robot description, xacro)
@@ -12,23 +12,15 @@
   <xacro:property name="M_PI" value="3.1415926535897931" />
   <xacro:property name="caster_offset_x" value="0.0" />
-  <xacro:property name="caster_offset_y" value="0.031" />
-  <xacro:property name="caster_offset_z" value="-0.11" />
-  <xacro:property name="caster_mass" value="0.0067" />
-  <xacro:property name="caster_collision_length" value="0.0176" />
-  <xacro:property name="caster_collision_radius" value="0.017" />
+  <xacro:property name="caster_offset_y" value="0.11" />
+  <xacro:property name="caster_offset_z" value="0.0" />
+  <xacro:property name="caster_mass" value="0.067" />
   <xacro:property name="wheel_offset_x" value="-0.132" />
   <xacro:property name="wheel_offset_y" value="0.022" />
   <xacro:property name="wheel_offset_z" value="-0.165" />
-  <xacro:property name="wheel_mass" value="0.38" />
-  <xacro:property name="wheel_length" value="0.0206" />
-  <xacro:property name="wheel_radius" value="0.0350" />
-  <xacro:property name="base_cg_x" value="0.0" />
-  <xacro:property name="base_cg_y" value="0.12403" />
-  <xacro:property name="base_cg_z" value="0.011243" />
+  <xacro:property name="wheel_mass" value="0.4" />
+  <xacro:property name="base_z" value="0.037" />
   <xacro:property name="base_mass" value="1.3083" />
-  <!-- simplified box collision geometry for base -->
   <xacro:property name="base_collision_length" value="0.10938" />
-  <xacro:property name="base_collision_radius" value="0.178" />
-  <xacro:property name="base_collision_z" value="0.05949" />
+  <xacro:property name="base_collision_radius" value="0.19" />
   <!-- Macro for aplha wheel (right/left)-->
   <!-- in typical convention param "reflect" equals +-1 to distinguish left from righ-->
@@ -64,5 +56,5 @@
         <origin xyz="0 0 0" rpy="${M_PI/2} 0 0" /> <!-- rotation because cyl. geom primitive has symmetry axis in +x direction -->
         <geometry>
-          <cylinder radius="${wheel_radius}" length="${wheel_length}" />
+          <mesh filename="package://alpha_description/meshes/chassis/wheel.STL" />
         </geometry>
       </collision>
@@ -82,5 +74,5 @@
       <inertial>
         <mass value="${caster_mass}"/>
-        <origin xyz="0 0 0" />
+        <origin xyz="0 0 0" rpy="0 0 0"/>
         <inertia ixx="7.34836188095286E-07"
                  ixy="-8.85813875476203E-23"
@@ -91,10 +83,7 @@
       </inertial>
       <visual>
-        <origin
-          xyz="0 0 0"
-          rpy="0 0 0" />
+        <origin xyz="0 0 0" rpy="0 0 0" />
         <geometry>
-          <mesh
-            filename="package://alpha_description/meshes/chassis/caster_body.STL" />
+          <mesh filename="package://alpha_description/meshes/chassis/caster_body.STL" />
         </geometry>
       </visual>
@@ -102,5 +91,5 @@
         <origin xyz="0 0 0" rpy="0 0 0" />
         <geometry>
-          <cylinder length="${caster_collision_length}" radius="${caster_collision_radius}"/>
+          <mesh filename="package://alpha_description/meshes/chassis/caster_body.STL" />
         </geometry>
       </collision>
@@ -161,5 +150,5 @@
       </inertial>
       <visual>
-        <origin xyz="0 0 0" rpy="0 0 0" />
+        <origin xyz="0 0 -0.031" rpy="${M_PI/2} 0 0" />
         <geometry>
           <mesh filename="package://alpha_description/meshes/chassis/base_plate.STL" />
@@ -168,5 +157,5 @@
       </visual>
       <collision>
-        <origin xyz="0 0 0" rpy="0 0 0" />
+        <origin xyz="0 0 ${base_collision_length/2}" rpy="0 0 0" />
         <geometry>
           <cylinder radius="${base_collision_radius}" length="${base_collision_length}" />
@@ -186,5 +175,5 @@
     </link>
     <joint name="${name}_footprint_joint" type="fixed">
-      <origin xyz="${base_cg_x} ${base_cg_y} ${base_cg_z}" rpy="${M_PI/2} 0 0" />
+      <origin xyz="0 0 ${base_z}" rpy="0 0 0" />
       <parent link="${name}_footprint"/>
       <child link="${name}_link" />
@@ -193,5 +182,5 @@
     <!-- caster macro -->
     <xacro:alpha_caster suffix="fl" parent="${name}_link" ref_position="${- M_PI/4}" >
-      <origin xyz="${caster_offset_x} ${caster_offset_y} ${caster_offset_z}" rpy="${-M_PI/2} 0 0" />
+      <origin xyz="${caster_offset_x} ${caster_offset_y} ${caster_offset_z}" rpy="${M_PI/2} 0 ${M_PI}" />
     </xacro:alpha_caster>
     <!-- gazebo extensions -->
