Commit message: alpha cad files added

File: simulation_module/alpha_description/robots/alpha_bot.urdf (robot description, URDF)
Before this commit: robot alpha, 8 links, 7 joints
Links:
- added link fl_caster_link, mass 0.0005236; collision mesh filename=package://alpha_description/meshes/chassis/caster_ball.STL; visual mesh filename=package://alpha_description/meshes/chassis/caster_ball.STL
- link base_link: mass 2.4 -> 1.3083; geometry collision cylinder length=0.10938 radius=0.178; visual mesh filename=package://alpha_description/meshes/chassis/base_plate.STL
- link fl_left_wheel_link: mass 0.01 -> 0.38; geometry collision cylinder length=0.0206 radius=0.035; visual mesh filename=package://alpha_description/meshes/chassis/wheel.STL
- link fl_right_wheel_link: mass 0.01 -> 0.38; geometry collision cylinder length=0.0206 radius=0.035; visual mesh filename=package://alpha_description/meshes/chassis/wheel.STL
- link fl_rotation_link: mass 0.01 -> 0.0067; geometry collision cylinder length=0.0176 radius=0.017; visual mesh filename=package://alpha_description/meshes/chassis/caster_body.STL
Joints:
- added joint fl_caster_joint: type fixed, parent fl_rotation_link, child fl_caster_link, origin xyz=0 -0.026 0 rpy=0 0 0, axis 0 0 0
- joint base_footprint_joint: axis (none) -> 0 0 0; origin xyz=0.0 0.0 0.065 rpy=0 0 0 -> xyz=0.0 0.12403 0.011243 rpy=1.57079632679 0 0
- joint fl_left_wheel_joint: axis 0 0 1 -> 0 0 -1; origin xyz=0 -0.14 0.0 rpy=1.57079632679 0 0 -> xyz=0.132 0.022 -0.165 rpy=1.57079632679 0 -1.57079632679
- joint fl_right_wheel_joint: origin xyz=0 0.14 0.0 rpy=1.57079632679 0 0 -> xyz=-0.132 0.022 -0.165 rpy=1.57079632679 0 1.57079632679
- joint fl_rotation_joint: origin xyz=0.0 0.0 -0.02 rpy=0 0 -1.57079632679 -> xyz=0.0 0.031 -0.11 rpy=-1.57079632679 0 0
- joint hokuyo_joint: origin xyz=0 0 0.332 rpy=0 0 0 -> xyz=0 0 0.332 rpy=0 0 1.57079632679

File: simulation_module/alpha_description/urdf/chassis/alpha_base.urdf.xacro (robot description, xacro)
@@ -12,19 +12,19 @@
   <xacro:property name="M_PI" value="3.1415926535897931" />
   <xacro:property name="caster_offset_x" value="0.0" />
-  <xacro:property name="caster_offset_y" value="0.0" />
-  <xacro:property name="caster_offset_z" value="-0.02" />
-  <xacro:property name="caster_mass" value="0.01" />
+  <xacro:property name="caster_offset_y" value="0.031" />
+  <xacro:property name="caster_offset_z" value="-0.11" />
+  <xacro:property name="caster_mass" value="0.0067" />
   <xacro:property name="caster_collision_length" value="0.0176" />
   <xacro:property name="caster_collision_radius" value="0.017" />
-  <xacro:property name="wheel_offset_y" value="0.14" />
-  <xacro:property name="wheel_offset_z" value="0.0" />
-  <xacro:property name="wheel_mass" value="0.01" />
+  <xacro:property name="wheel_offset_x" value="-0.132" />
+  <xacro:property name="wheel_offset_y" value="0.022" />
+  <xacro:property name="wheel_offset_z" value="-0.165" />
+  <xacro:property name="wheel_mass" value="0.38" />
   <xacro:property name="wheel_length" value="0.0206" />
   <xacro:property name="wheel_radius" value="0.0350" />
   <xacro:property name="base_cg_x" value="0.0" />
-  <xacro:property name="base_cg_y" value="0.0" />
-  <xacro:property name="base_cg_z" value="0.065" />
-  <xacro:property name="base_visual_offset" value="-0.095" />
-  <xacro:property name="base_mass" value="2.4" />
+  <xacro:property name="base_cg_y" value="0.12403" />
+  <xacro:property name="base_cg_z" value="0.011243" />
+  <xacro:property name="base_mass" value="1.3083" />
   <!-- simplified box collision geometry for base -->
   <xacro:property name="base_collision_length" value="0.10938" />
@@ -35,9 +35,9 @@
   <xacro:macro name="alpha_wheel" params="suffix parent reflect">
     <joint name="${parent}_${suffix}_wheel_joint" type="continuous">
-      <axis xyz="0 0 1" />
+      <axis xyz="0 0 ${reflect * 1}" />
       <limit effort="18" velocity="1.5"/>
       <safety_controller  k_velocity="1" />
       <dynamics damping="1.0" friction="0.0" />
-      <origin xyz="0 ${reflect * wheel_offset_y} ${wheel_offset_z}" rpy="${M_PI/2} 0 0" />
+      <origin xyz="${reflect * wheel_offset_x} ${wheel_offset_y} ${wheel_offset_z}" rpy="${M_PI/2} 0 ${reflect * M_PI/2}" />
       <parent link="${parent}_rotation_link"/>
       <child link="${parent}_${suffix}_wheel_link"/>
@@ -47,12 +47,15 @@
         <mass value="${wheel_mass}" />
         <origin xyz="0 0 0" />
-        <inertia  ixx="0.001" ixy="0.0" ixz="0.0"
-                  iyy="0.001" iyz="0.0"
-                  izz="0.001" />
-      </inertial>
-      <visual>
-        <origin xyz="0 0 0" rpy="0 0 0" />
-        <geometry>
-          <mesh filename="package://alpha_description/meshes/chassis/wheel.dae" />
+        <inertia ixx="0.00027992"
+                 ixy="-1.1223E-19"
+                 ixz="2.6988E-20"
+                 iyy="0.00027992"
+                 iyz="8.6881E-21"
+                 izz="0.00045332"/>
+      </inertial>
+      <visual>
+        <origin xyz="0 0 0" rpy="0 0 0" />
+        <geometry>
+          <mesh filename="package://alpha_description/meshes/chassis/wheel.STL" />
         </geometry>
         <material name="Black" />
@@ -72,5 +75,5 @@
   <xacro:macro name="alpha_caster_hub" params="suffix parent *origin ref_position" >
     <joint name="${suffix}_rotation_joint" type="fixed">
-      <origin xyz="${caster_offset_x} ${caster_offset_y} ${caster_offset_z}" rpy="0 0 ${-M_PI/2}"/>
+      <xacro:insert_block name="origin" />
       <parent link="${parent}"/>
       <child link="${suffix}_rotation_link" />
@@ -80,8 +83,20 @@
         <mass value="${caster_mass}"/>
         <origin xyz="0 0 0" />
-        <inertia ixx="0.001" ixy="0.0" ixz="0.0"
-                 iyy="0.001" iyz="0.0"
-                 izz="0.001" />
-      </inertial>
+        <inertia ixx="7.34836188095286E-07"
+                 ixy="-8.85813875476203E-23"
+                 ixz="-2.27179291546233E-23"
+                 iyy="5.26473063708137E-07"
+                 iyz="-1.32876082683251E-22"
+                 izz="7.34836188095287E-07" />
+      </inertial>
+      <visual>
+        <origin
+          xyz="0 0 0"
+          rpy="0 0 0" />
+        <geometry>
+          <mesh
+            filename="package://alpha_description/meshes/chassis/caster_body.STL" />
+        </geometry>
+      </visual>
       <collision>
         <origin xyz="0 0 0" rpy="0 0 0" />
@@ -91,4 +106,34 @@
       </collision>
     </link>
+    <link name="${suffix}_caster_link">
+      <inertial>
+        <origin xyz="0 0 0" rpy="0 0 0" />
+        <mass value="0.0005236" />
+        <inertia ixx="5.236E-09"
+                 ixy="1.551E-25"
+                 ixz="1.034E-25"
+                 iyy="5.236E-09"
+                 iyz="6.2039E-25"
+                 izz="5.236E-09" />
+      </inertial>
+      <visual>
+        <origin xyz="0 0 0" rpy="0 0 0" />
+        <geometry>
+          <mesh filename="package://alpha_description/meshes/chassis/caster_ball.STL" />
+        </geometry>
+      </visual>
+      <collision>
+        <origin xyz="0 0 0" rpy="0 0 0" />
+        <geometry>
+          <mesh filename="package://alpha_description/meshes/chassis/caster_ball.STL" />
+        </geometry>
+      </collision>
+    </link>
+    <joint name="${suffix}_caster_joint" type="fixed">
+      <origin xyz="0 -0.026 0" rpy="0 0 0" />
+      <parent link="${suffix}_rotation_link" />
+      <child link="${suffix}_caster_link" />
+      <axis xyz="0 0 0" />
+    </joint>
     <!-- extensions -->
     <xacro:alpha_caster_transmission suffix="${suffix}" />
@@ -110,13 +155,13 @@
       <inertial>
         <mass value="${base_mass}" />
-        <origin xyz="0 0 0" />
-        <inertia ixx="0.019995" ixy="0.0" ixz="0.0"
-                 iyy="0.019995" iyz="0.0"
-                 izz="0.03675" />
-      </inertial>
-      <visual>
-        <origin xyz="0 0 ${base_visual_offset}" rpy="0 0 0" />
-        <geometry>
-          <mesh filename="package://alpha_description/meshes/chassis/base_plate.dae" />
+        <origin xyz="0 0 0" rpy="0 0 0"/>
+        <inertia ixx="0.016994" ixy="1.2142E-05" ixz="-1.5304E-05"
+                 iyy="0.015814" iyz="0.00078225"
+                 izz="0.022766" />
+      </inertial>
+      <visual>
+        <origin xyz="0 0 0" rpy="0 0 0" />
+        <geometry>
+          <mesh filename="package://alpha_description/meshes/chassis/base_plate.STL" />
         </geometry>
         <material name="White" />
@@ -141,11 +186,12 @@
     </link>
     <joint name="${name}_footprint_joint" type="fixed">
-      <origin xyz="${base_cg_x} ${base_cg_y} ${base_cg_z}" rpy="0 0 ${-M_PI/2}" />
+      <origin xyz="${base_cg_x} ${base_cg_y} ${base_cg_z}" rpy="${M_PI/2} 0 0" />
       <parent link="${name}_footprint"/>
       <child link="${name}_link" />
+      <axis xyz="0 0 0" />
     </joint>
     <!-- caster macro -->
     <xacro:alpha_caster suffix="fl" parent="${name}_link" ref_position="${- M_PI/4}" >
-      <origin xyz="${caster_offset_x} ${caster_offset_y} ${caster_offset_z}" rpy="0 0 0" />
+      <origin xyz="${caster_offset_x} ${caster_offset_y} ${caster_offset_z}" rpy="${-M_PI/2} 0 0" />
     </xacro:alpha_caster>
     <!-- gazebo extensions -->

Commit message: updated .urdf file

File: simulation_module/alpha_description/robots/alpha_bot.urdf (robot description, URDF)
Before this commit: robot alpha, 9 links, 8 joints
Joints:
- joint base_footprint_joint: origin xyz=0 0 0.037 rpy=0 0 -1.57079632679 -> xyz=0 0 0.0365 rpy=0 0 -1.57079632679
