Commit message: color to wheels [unresolved]

File: simulation_module/alpha_description/urdf/chassis/alpha_base.urdf.xacro (robot description, xacro)
@@ -56,5 +56,5 @@
           <mesh filename="package://alpha_description/meshes/chassis/wheel.dae" />
         </geometry>
-        <material name="Wheel_${suffix}" />
+        <material name="Black" />
       </visual>
       <collision>

Commit message: dummy link added for base_footprint

File: simulation_module/alpha_description/urdf/chassis/alpha_base.urdf.xacro (robot description, xacro)
@@ -132,11 +132,4 @@
          navigation stack dedpends on this frame -->
     <link name="${name}_footprint">
-      <inertial>
-        <mass value="1.0" />
-        <origin xyz="0 0 0" />
-        <inertia ixx="0.019995" ixy="0.0" ixz="0.0"
-                 iyy="0.019995" iyz="0.0"
-                 izz="0.03675" />
-      </inertial>
       <visual>
         <origin xyz="0 0 0" rpy="0 0 0" />
@@ -146,12 +139,4 @@
         <material name="White" />
       </visual>
-      <collision>
-        <!-- represent base collision with a simple rectangular model, positioned by base_size_z s.t. top
-             surface of the collision box matches the top surface of the alpha base -->
-        <origin xyz="0 0 ${base_collision_z/2}" rpy="0 0 0" />
-        <geometry>
-          <box size="0.001 0.001 0.001" />
-        </geometry>
-      </collision>
     </link>
     <joint name="${name}_footprint_joint" type="fixed">

Commit message: odom direction fixed

File: simulation_module/alpha_description/urdf/chassis/alpha_base.urdf.xacro (robot description, xacro)
@@ -141,5 +141,5 @@
     </link>
     <joint name="${name}_footprint_joint" type="fixed">
-      <origin xyz="${base_cg_x} ${base_cg_y} ${base_cg_z}" rpy="0 0 0" />
+      <origin xyz="${base_cg_x} ${base_cg_y} ${base_cg_z}" rpy="0 0 ${-M_PI/2}" />
       <parent link="${name}_footprint"/>
       <child link="${name}_link" />

Commit message: slam rviz added

File: simulation_module/alpha_description/urdf/chassis/alpha_base.urdf.xacro (robot description, xacro)
@@ -19,5 +19,5 @@
   <xacro:property name="wheel_offset_z" value="-0.165" />
   <xacro:property name="wheel_mass" value="1.0" />
-  <xacro:property name="base_z" value="0.037" />
+  <xacro:property name="base_z" value="0.0365" />
   <xacro:property name="base_mass" value="8.5" />
   <xacro:property name="base_collision_length" value="0.10938" />
