Commit message: transmission corrected

File: simulation_module/alpha_description/urdf/chassis/alpha_base.gazebo.xacro (robot description, xacro)
@@ -11,19 +11,22 @@
       <kd  value="100.0" />
       <maxVel  value="1.0" />
-      <minDepth  value="0.001" />
+      <minDepth  value="0.0" />
+      <material>Gazebo/Black</material>
     </gazebo>
   </xacro:macro>
   <xacro:macro name="alpha_caster_gazebo" params="suffix">
-    <gazebo reference="${suffix}_caster_rotation_link">
-      <mu1 value="0.0" />
-      <mu2 value="0.0" />
+    <gazebo reference="${suffix}_caster_link">
+      <mu1 value="0.2" />
+      <mu2 value="0.2" />
       <kp value="1000000.0" />
       <kd value="100.0" />
-      <minDepth value="0.001" />
       <maxVel value="1.0" />
+      <minDepth value="0.0" />
+      <material>Gazebo/Black</material>
     </gazebo>
   </xacro:macro>
   <xacro:macro name="alpha_base_gazebo" params="name">
     <gazebo reference="${name}_link">
+      <material>Gazebo/Grey</material>
       <plugin name="p3d_base_controller" filename="libgazebo_ros_p3d.so">
         <alwaysOn>true</alwaysOn>
@@ -41,9 +44,9 @@
         <robotNamespace>/</robotNamespace>
         <alwaysOn>true</alwaysOn>
-        <updateRate>20</updateRate>
+        <updateRate>100.0</updateRate>
         <leftJoint>fl_left_wheel_joint</leftJoint>
         <rightJoint>fl_right_wheel_joint</rightJoint>
         <wheelSeparation>0.30</wheelSeparation>
-        <wheelDiameter>0.09</wheelDiameter>
+        <wheelDiameter>0.07</wheelDiameter>
         <wheelTorque>20</wheelTorque>
         <wheelAcceleration>0</wheelAcceleration>
@@ -53,5 +56,5 @@
         <robotBaseFrame>${name}_footprint</robotBaseFrame>
         <legacyMode>true</legacyMode>
-        <publishWheelTF>true</publishWheelTF>
+        <publishWheelTF>false</publishWheelTF>
         <publishWheelJointState>true</publishWheelJointState>
         <publishTf>1</publishTf>

File: simulation_module/alpha_description/urdf/chassis/alpha_base.urdf.xacro (robot description, xacro)
@@ -14,11 +14,11 @@
   <xacro:property name="caster_offset_y" value="0.11" />
   <xacro:property name="caster_offset_z" value="0.0" />
-  <xacro:property name="caster_mass" value="0.067" />
+  <xacro:property name="caster_mass" value="0.2" />
   <xacro:property name="wheel_offset_x" value="-0.132" />
   <xacro:property name="wheel_offset_y" value="0.022" />
   <xacro:property name="wheel_offset_z" value="-0.165" />
-  <xacro:property name="wheel_mass" value="0.4" />
+  <xacro:property name="wheel_mass" value="1.0" />
   <xacro:property name="base_z" value="0.037" />
-  <xacro:property name="base_mass" value="1.3083" />
+  <xacro:property name="base_mass" value="8.5" />
   <xacro:property name="base_collision_length" value="0.10938" />
   <xacro:property name="base_collision_radius" value="0.19" />
@@ -54,5 +54,5 @@
       </visual>
       <collision>
-        <origin xyz="0 0 0" rpy="${M_PI/2} 0 0" /> <!-- rotation because cyl. geom primitive has symmetry axis in +x direction -->
+        <origin xyz="0 0 0" rpy="0 0 0" /> <!-- rotation because cyl. geom primitive has symmetry axis in +x direction -->
         <geometry>
           <mesh filename="package://alpha_description/meshes/chassis/wheel.STL" />
@@ -87,4 +87,5 @@
           <mesh filename="package://alpha_description/meshes/chassis/caster_body.STL" />
         </geometry>
+        <material name="Black" />
       </visual>
       <collision>
@@ -145,6 +146,9 @@
         <mass value="${base_mass}" />
         <origin xyz="0 0 0" rpy="0 0 0"/>
-        <inertia ixx="0.016994" ixy="1.2142E-05" ixz="-1.5304E-05"
-                 iyy="0.015814" iyz="0.00078225"
+        <inertia ixx="0.016994"
+                 ixy="1.2142E-05"
+                 ixz="-1.5304E-05"
+                 iyy="0.015814"
+                 iyz="0.00078225"
                  izz="0.022766" />
       </inertial>
@@ -175,5 +179,5 @@
     </link>
     <joint name="${name}_footprint_joint" type="fixed">
-      <origin xyz="0 0 ${base_z}" rpy="0 0 0" />
+      <origin xyz="0 0 ${base_z}" rpy="0 0 ${-M_PI/2}" />
       <parent link="${name}_footprint"/>
       <child link="${name}_link" />

File: simulation_module/alpha_description/urdf/sensors/kinect/v2/kinect.urdf.xacro (robot description, xacro)
@@ -20,5 +20,5 @@
     <link name="${name}_frame">
       <inertial>
-        <mass value="0.1" />
+        <mass value="1.4" />
         <origin xyz="0 0 0" rpy="0 0 0"/>
         <inertia ixx="0.01"  ixy="0.0"  ixz="0.0"

Commit message: gmapping with teleop launch file created

File: simulation_module/alpha_description/urdf/chassis/alpha_base.gazebo.xacro (robot description, xacro)
@@ -1,7 +1,7 @@
 <?xml version="1.0"?>
 <robot xmlns:xacro="http://ros.org/wiki/xacro">
-  <xacro:property name="base_link_wheel_seperation" value="0.30" />
-  <xacro:property name="base_link_wheel_diameter" value="0.09" />
-  <xacro:property name="base_link_wheel_torque" value="0.01" />
+  <xacro:property name="base_link_wheel_seperation" value="0.308" />
+  <xacro:property name="base_link_wheel_diameter" value="0.106" />
+  <xacro:property name="base_link_wheel_torque" value="20" />
   <xacro:macro name="alpha_wheel_gazebo" params="suffix parent">
     <gazebo reference="${parent}_${suffix}_wheel_link">
@@ -47,7 +47,7 @@
         <leftJoint>fl_left_wheel_joint</leftJoint>
         <rightJoint>fl_right_wheel_joint</rightJoint>
-        <wheelSeparation>0.308</wheelSeparation>
-        <wheelDiameter>0.106/wheelDiameter>
-        <wheelTorque>20</wheelTorque>
+        <wheelSeparation>${base_link_wheel_seperation}</wheelSeparation>
+        <wheelDiameter>${base_link_wheel_diameter}</wheelDiameter>
+        <wheelTorque>${base_link_wheel_torque}</wheelTorque>
         <wheelAcceleration>0</wheelAcceleration>
         <commandTopic>cmd_vel</commandTopic>

Commit message: changed gazebo topics

File: simulation_module/alpha_description/urdf/chassis/alpha_base.gazebo.xacro (robot description, xacro)
@@ -26,5 +26,5 @@
     </gazebo>
   </xacro:macro>
-  <xacro:macro name="alpha_base_gazebo" params="name">
+  <xacro:macro name="alpha_base_gazebo" params="name ns:=/">
     <gazebo>
       <material>Gazebo/Grey</material>
@@ -42,5 +42,5 @@
     <gazebo>
       <plugin name="differential_drive_controller" filename="libgazebo_ros_diff_drive.so">
-        <robotNamespace>/</robotNamespace>
+        <robotNamespace>${ns}</robotNamespace>
         <alwaysOn>true</alwaysOn>
         <updateRate>100.0</updateRate>

File: simulation_module/alpha_description/urdf/sensors/hokuyo_laser/hokuyo_lx30_laser.gazebo.xacro (robot description, xacro)
@@ -1,5 +1,5 @@
 <?xml version="1.0"?>
 <robot xmlns:xacro="http://ros.org/wiki/xacro">
-  <xacro:macro name="hokuyo_lx30_laser_gazebo" params="name ros_topic update_rate min_angle max_angle">
+  <xacro:macro name="hokuyo_lx30_laser_gazebo" params="name ros_topic update_rate min_angle max_angle ns:=/ ">
     <gazebo reference="${name}_frame">
       <sensor type="ray" name="${name}">
@@ -33,5 +33,5 @@
         </ray>
         <plugin name="gazebo_ros_${name}_controller" filename="libgazebo_ros_laser.so">
-          <robotNamespace>/</robotNamespace>
+          <robotNamespace>${ns}</robotNamespace>
           <gaussianNoise>0.005</gaussianNoise>
           <alwaysOn>true</alwaysOn>

File: simulation_module/alpha_description/urdf/sensors/kinect/v2/kinect.gazebo.xacro (robot description, xacro)
@@ -1,5 +1,5 @@
 <?xml version="1.0"?>
 <robot xmlns:xacro="http://ros.org/wiki/xacro">
-  <xacro:macro name="kinect_camera_gazebo" params="name">
+  <xacro:macro name="kinect_camera_gazebo" params="name ns:=/ ">
     <gazebo reference="${name}_frame">
       <sensor type="depth" name="${name}_frame_sensor">
@@ -19,13 +19,13 @@
         </camera>
         <plugin name="${name}_frame_controller" filename="libgazebo_ros_openni_kinect.so">
-          <robotNamespace>/</robotNamespace>
+          <robotNamespace>${ns}</robotNamespace>
           <alwaysOn>true</alwaysOn>
           <updateRate>20.0</updateRate>
           <cameraName>${name}</cameraName>
-          <imageTopicName>${name}/ir/image_raw</imageTopicName>
-          <cameraInfoTopicName>${name}/ir/camera_info</cameraInfoTopicName>
-          <depthImageTopicName>${name}/depth/image_raw</depthImageTopicName>
-          <depthImageCameraInfoTopicName>${name}/depth/camera_info</depthImageCameraInfoTopicName>
-          <pointCloudTopicName>${name}/depth/points</pointCloudTopicName>
+          <imageTopicName>scene/image_raw</imageTopicName>
+          <cameraInfoTopicName>scene/camera_info</cameraInfoTopicName>
+          <depthImageTopicName>depth/image_raw</depthImageTopicName>
+          <depthImageCameraInfoTopicName>depth/camera_info</depthImageCameraInfoTopicName>
+          <pointCloudTopicName>depth/points</pointCloudTopicName>
           <frameName>${name}_optical_frame</frameName>
           <pointCloudCutoff>0.5</pointCloudCutoff>

File: simulation_module/alpha_description/urdf/sensors/kinect/xbox360/kinect.gazebo.xacro (robot description, xacro)
@@ -1,5 +1,5 @@
 <?xml version="1.0"?>
 <robot xmlns:xacro="http://ros.org/wiki/xacro">
-  <xacro:macro name="kinect_camera_gazebo" params="name">
+  <xacro:macro name="kinect_camera_gazebo" params="name ns:=/ ">
     <gazebo reference="${name}_frame">
       <sensor type="depth" name="${name}_frame_sensor">
@@ -19,13 +19,13 @@
         </camera>
         <plugin name="${name}_frame_controller" filename="libgazebo_ros_openni_kinect.so">
-          <robotNamespace>/</robotNamespace>
+          <robotNamespace>${ns}</robotNamespace>
           <alwaysOn>true</alwaysOn>
           <updateRate>20.0</updateRate>
           <cameraName>${name}</cameraName>
-          <imageTopicName>${name}/ir/image_raw</imageTopicName>
-          <cameraInfoTopicName>${name}/ir/camera_info</cameraInfoTopicName>
-          <depthImageTopicName>${name}/depth/image_raw</depthImageTopicName>
-          <depthImageCameraInfoTopicName>${name}/depth/camera_info</depthImageCameraInfoTopicName>
-          <pointCloudTopicName>${name}/depth/points</pointCloudTopicName>
+          <imageTopicName>scene/image_raw</imageTopicName>
+          <cameraInfoTopicName>scene/camera_info</cameraInfoTopicName>
+          <depthImageTopicName>depth/image_raw</depthImageTopicName>
+          <depthImageCameraInfoTopicName>depth/camera_info</depthImageCameraInfoTopicName>
+          <pointCloudTopicName>depth/points</pointCloudTopicName>
           <frameName>${name}_optical_frame</frameName>
           <pointCloudCutoff>0.5</pointCloudCutoff>
@@ -61,9 +61,9 @@
           <updateRate>20.0</updateRate>
           <cameraName>${name}</cameraName>
-          <imageTopicName>${name}/rgb/image_raw</imageTopicName>
-          <cameraInfoTopicName>${name}/rgb/camera_info</cameraInfoTopicName>
-          <depthImageTopicName>${name}/depth/image_raw</depthImageTopicName>
-          <depthImageCameraInfoTopicName>${name}/depth/camera_info</depthImageCameraInfoTopicName>
-          <pointCloudTopicName>${name}/rgb/points</pointCloudTopicName>
+          <imageTopicName>/rgb/image_raw</imageTopicName>
+          <cameraInfoTopicName>/rgb/camera_info</cameraInfoTopicName>
+          <depthImageTopicName>/depth/image_raw</depthImageTopicName>
+          <depthImageCameraInfoTopicName>/depth/camera_info</depthImageCameraInfoTopicName>
+          <pointCloudTopicName>/rgb/points</pointCloudTopicName>
           <frameName>${name}_optical_frame</frameName>
           <pointCloudCutoff>0.5</pointCloudCutoff>
